Commit message: sdf file

File: src/my_robot/urdf/robot.urdf (robot description, URDF)
Before this commit: robot my_robot, 10 links, 9 joints
Links:
- link base_link: mass 60.1 -> 500.1
- link link_chair: mass 0.0383122914433503 -> 10
- link link_f_l: mass 0.135994744058479 -> 30
- link link_f_l_w: mass 2.57224227872115 -> 50
- link link_f_r: mass 0.135994744058479 -> 30
- link link_f_r_w: mass 2.57224227872849 -> 50
- link link_l_w: mass 5.33437190224873 -> 80
- link link_r_w: mass 5.33437190113988 -> 80
- link link_w: mass 0.00423185835861639 -> 5
Joints:
- joint world_to_base: origin xyz=0 0 0 rpy=0 0 0 -> xyz=0 0 1 rpy=0 0 0
