Commit message: rf-detr

File: src/my_robot/urdf/fito.urdf (robot description, URDF)
Before this commit: robot my_robot, 18 links, 17 joints
Joints:
- joint front_wheels_base_to_depth_camera: origin xyz=-0.08 0 0 rpy=1.57 0 -1.57 -> xyz=-0.06 0 0 rpy=1.0 3.14 -1.57

Commit message: gps

File: src/my_robot/urdf/fito.urdf (robot description, URDF)
Before this commit: robot my_robot, 18 links, 17 joints
Links:
- added link gps_link, mass 0.1; collision box size=0.07 0.05 0.05; visual box size=0.07 0.05 0.05
Joints:
- added joint gps_joint: type fixed, parent base_link, child gps_link, origin xyz=0 0 0.07 rpy=0 0 0

Commit message: gps update

File: src/my_robot/urdf/fito.urdf (robot description, URDF)
Before this commit: robot my_robot, 19 links, 18 joints
Links:
- removed link fito_world
- added link base_footprint
Joints:
- joint base_joint: parent fito_world -> base_footprint

Commit message: minor changes in urdf odometry

File: src/my_robot/urdf/fito.urdf (robot description, URDF)
Before this commit: robot my_robot, 19 links, 18 joints
Joints:
- joint base_joint: origin xyz=0 0 0 rpy=0 0 0 -> xyz=0 0 0.74 rpy=0 0 3.14

Commit message: urdf setting for lane following

File: src/my_robot/urdf/fito.urdf (robot description, URDF)
Before this commit: robot my_robot, 19 links, 18 joints
Joints:
- joint base_joint: origin xyz=0 0 0.74 rpy=0 0 3.14 -> xyz=0 0 0.74 rpy=0 0 3.14159265358979323846159265358979323846
- joint base_link_to_wheeling_mech: limit lower=-0.4 upper=0.4 effort=3000.0 velocity=0.5 -> lower=-0.3 upper=0.3 effort=3000.0 velocity=1
- joint front_wheels_base_to_depth_camera: origin xyz=-0.06 0 0 rpy=1.0 3.14 -1.57 -> xyz=-2.3 0 1 rpy=0 0 0; parent front_wheels_base -> base_link

Commit message: line correction

File: src/my_robot/urdf/fito.urdf (robot description, URDF)
Before this commit: robot my_robot, 19 links, 18 joints
Joints:
- joint front_wheels_base_to_depth_camera: axis (none) -> 0 1 0; limit (none) -> lower=0.0 upper=2.09 effort=10 velocity=1; type fixed -> revolute
