Commit message: ros2_control_update

File: install/my_robot/share/my_robot/urdf/robot.xacro (robot description, xacro)
@@ -40,5 +40,5 @@
   </xacro:macro>
   <!-- Wheel macro -->
-  <xacro:macro name="wheel_assembly" params="prefix parent xyz rpy steering_limits is_driven:=false">
+  <xacro:macro name="wheel_assembly" params="prefix parent xyz rpy steering_lower steering_upper is_driven:=false">
     <!-- Steering link (f_l или f_r) -->
     <xacro:standard_link
@@ -57,5 +57,5 @@
       <origin xyz="${xyz}" rpy="${rpy}"/>
       <axis xyz="0 1 0"/>
-      <limit lower="${steering_limits[0]}" upper="${steering_limits[1]}" effort="100" velocity="1.0"/>
+      <limit lower="${steering_lower}" upper="${steering_upper}" effort="100" velocity="1.0"/>
     </joint>
     <!-- Wheel (f_l_w или f_r_w) -->
@@ -149,7 +149,7 @@
   <!-- Front wheels (steerable) -->
   <xacro:wheel_assembly prefix="f_r" parent="base_link"
-    xyz="-0.11936 0.03 -0.083652" rpy="1.5708 0 3.1403" steering_limits="-0.5 0.5"/>
+    xyz="-0.11936 0.03 -0.083652" rpy="1.5708 0 3.1403" steering_lower="-1.57" steering_upper="1.57"/>
   <xacro:wheel_assembly prefix="f_l" parent="base_link"
-    xyz="-0.11936 -0.03 -0.083652" rpy="1.5708 0 -0.0013373" steering_limits="-0.5 0.5"/>
+    xyz="-0.11936 -0.03 -0.083652" rpy="1.5708 0 -0.0013373" steering_lower="-1.57" steering_upper="1.57"/>
   <!-- Rear wheels (driven) -->
   <xacro:rear_wheel_assembly prefix="r" parent="base_link" is_driven="true"
@@ -185,7 +185,7 @@
   <!-- ==================== ROS 2 CONTROL ==================== -->
   <xacro:if value="$(arg use_gazebo)">
-    <ros2_control name="GazeboSystem" type="system">
+    <ros2_control name="RobotController" type="system">
       <hardware>
-        <plugin>gazebo_ros2_control/GazeboSystem</plugin>
+        <plugin>gz_ros2_control/GazeboSimSystem</plugin>
       </hardware>
       <!-- Wheel motors (velocity control) -->
@@ -209,5 +209,5 @@
       <joint name="joint_f_r">
         <command_interface name="position">
-          <param name="min">-0.5</param>
+          <param name="min">0</param>
           <param name="max">0.5</param>
         </command_interface>
@@ -216,5 +216,5 @@
       <joint name="joint_f_l">
         <command_interface name="position">
-          <param name="min">-0.5</param>
+          <param name="min">0</param>
           <param name="max">0.5</param>
         </command_interface>
@@ -227,5 +227,5 @@
     <!-- ROS 2 Control plugin -->
     <gazebo>
-      <plugin name="gazebo_ros2_control" filename="libgazebo_ros2_control.so">
+      <plugin name="gz_ros2_control::GazeboSimROS2ControlPlugin" filename="libgz_ros2_control-system.so">
         <parameters>$(find my_robot)/config/controllers.yaml</parameters>
       </plugin>

File: install/my_robot/share/my_robot/urdf/robot2.urdf (robot description, URDF)
Before this commit: robot my_robot, 10 links, 9 joints
Joints:
- joint joint_f_l: limit lower=- upper=0 effort=100 velocity=1.0 -> lower=-1 upper=0 effort=100 velocity=1.0
- joint joint_f_r: limit lower=- upper=0 effort=100 velocity=1.0 -> lower=-1 upper=0 effort=100 velocity=1.0

Commit message: IT_DOESNT_FREEZE

File: install/my_robot/share/my_robot/urdf/robot.xacro (robot description, xacro)
@@ -130,5 +130,5 @@
   <!-- ==================== ROBOT STRUCTURE ==================== -->
   <!-- World link -->
-  <link name="world"/>
+  <link name="car_world"/>
   <!-- Base link -->
   <xacro:standard_link
@@ -143,5 +143,5 @@
   </xacro:standard_link>
   <joint name="world_to_base" type="fixed">
-    <parent link="world"/>
+    <parent link="car_world"/>
     <child link="base_link"/>
     <origin xyz="0 0 1" rpy="0 0 0"/>
@@ -185,10 +185,9 @@
   <!-- ==================== ROS 2 CONTROL ==================== -->
   <xacro:if value="$(arg use_gazebo)">
-    <ros2_control name="RobotController" type="system">
+    <ros2_control name="GazeboSystem" type="system">
       <hardware>
         <plugin>gz_ros2_control/GazeboSimSystem</plugin>
       </hardware>
-      <!-- Wheel motors (velocity control) -->
-      <joint name="joint_r_w">
+      <joint name="joint_l_w">
         <command_interface name="velocity">
           <param name="min">-10</param>
@@ -198,5 +197,6 @@
         <state_interface name="velocity"/>
       </joint>
-      <joint name="joint_l_w">
+      <!-- Wheel motors (velocity control) -->
+      <joint name="joint_r_w">
         <command_interface name="velocity">
           <param name="min">-10</param>
@@ -230,4 +230,26 @@
         <parameters>$(find my_robot)/config/controllers.yaml</parameters>
       </plugin>
+              <!--plugin name="gz::sim::systems::DiffDrive" filename="gz-sim-diff-drive-system">
+            <right_joint>joint_r_w</right_joint>
+            <wheel_separation>0.297</wheel_separation>
+            <wheel_radius>0.033</wheel_radius>
+            <max_linear_acceleration>0.33</max_linear_acceleration>
+            <topic>cmd_vel</topic>
+            <frame_id>odom</frame_id>
+            <child_frame_id>base_link</child_frame_id>
+            <odom_topic>odom</odom_topic>
+            <odom_publisher_frequency>30</odom_publisher_frequency>
+            <tf_topic>/tf</tf_topic>
+        </plugin> -->
+        <!-- <plugin filename="gz-sim-joint-state-publisher-system"
+            name="gz::sim::systems::JointStatePublisher">
+            <topic>joint_states</topic>
+            <joint_name>joint_f_r</joint_name>
+            <joint_name>joint_f_l</joint_name>
+            <joint_name>joint_r_w</joint_name>
+            <joint_name>joint_l_w</joint_name>
+            <joint_name>joint_f_r_w</joint_name>
+            <joint_name>joint_f_l_w</joint_name>
+        </plugin> -->
     </gazebo>
     <!-- Default material -->

Commit message: lidar

File: install/my_robot/share/my_robot/urdf/robot.xacro (robot description, xacro)
@@ -206,4 +206,20 @@
         <state_interface name="velocity"/>
       </joint>
+      <joint name="joint_f_l_w">
+        <command_interface name="velocity">
+          <param name="min">-10</param>
+          <param name="max">10</param>
+        </command_interface>
+        <state_interface name="position"/>
+        <state_interface name="velocity"/>
+      </joint>
+      <joint name="joint_f_r_w">
+        <command_interface name="velocity">
+          <param name="min">-10</param>
+          <param name="max">10</param>
+        </command_interface>
+        <state_interface name="position"/>
+        <state_interface name="velocity"/>
+      </joint>
       <!-- Steering mechanisms (position control) -->
       <joint name="joint_f_r">
@@ -213,4 +229,5 @@
         </command_interface>
         <state_interface name="position"/>
+        <state_interface name="velocity"/>
       </joint>
       <joint name="joint_f_l">
@@ -220,4 +237,5 @@
         </command_interface>
         <state_interface name="position"/>
+        <state_interface name="velocity"/>
       </joint>
     </ros2_control>
