Commit message: joy_control

File: install/my_robot/share/my_robot/urdf/fito.urdf (robot description, URDF)
Before this commit: robot my_robot, 16 links, 15 joints
Links:
- added link odom
Joints:
- added joint base_odom_joint: type floating, parent fito_world, child odom, origin xyz=0 0 0 rpy=0 0 0
- joint base_joint: origin xyz=0 0.03266198015150823 0 rpy=0 0 0 -> xyz=0 0 0 rpy=0 0 0

File: src/my_robot/urdf/fito.urdf (robot description, URDF)
Before this commit: robot my_robot, 16 links, 15 joints
Joints:
- joint base_joint: origin xyz=0 0.03266198015150823 0 rpy=0 0 0 -> xyz=0 0 0 rpy=0 0 0

Commit message: odom_update

File: install/my_robot/share/my_robot/urdf/fito.urdf (robot description, URDF)
Before this commit: robot my_robot, 17 links, 16 joints
Links:
- removed link odom
- added link base_footprint
Joints:
- removed joint base_odom_joint
- added joint base_footprint_joint: type fixed, parent fito_world, child base_footprint, origin xyz=0 0 0 rpy=0 0 0

File: src/my_robot/urdf/fito.urdf (robot description, URDF)
Before this commit: robot my_robot, 16 links, 15 joints
Links:
- added link base_footprint
Joints:
- added joint base_footprint_joint: type fixed, parent fito_world, child base_footprint, origin xyz=0 0 0 rpy=0 0 0

Commit message: added rtab-slam

File: install/my_robot/share/my_robot/urdf/fito.urdf (robot description, URDF)
Before this commit: robot my_robot, 17 links, 16 joints
Links:
- removed link base_footprint
- added link depth_camera_link, mass 0.1; collision box size=0.07 0.05 0.05; visual box size=0.07 0.05 0.05
- added link imu_link, mass 0.1; collision box size=0.07 0.05 0.05; visual box size=0.07 0.05 0.05
Joints:
- removed joint base_footprint_joint
- added joint front_wheels_base_to_depth_camera: type fixed, parent front_wheels_base, child depth_camera_link, origin xyz=-0.08 0 0 rpy=1.57 0 -1.57
- added joint imu_joint: type fixed, parent base_link, child imu_link, origin xyz=0.1 0 0.1 rpy=0 0 0
